File: development/arena_12-12_w_vreg/ni/ni_arena_12-12_v0p1/ni_arena_12-12.kicad_sch (KiCad schematic)
At the start: 0 parts

Commit message: double checking, adding BOM
Other:
- company: (none) -> IORodeo for Reiserlab @ Janelia
- title: (none) -> 12-12 NI G4.1 Arena Modular LED Display
