File: development/arena_12-12_w_vreg/ni/ni_arena_12-12_v0p1/panel_headers.kicad_sch (KiCad schematic)
At the start: 15 parts, among them P1 CONN15, P10 CONN15, P11 CONN15, P12 CONN15, P2 CONN15, P3 CONN15, P4 CONN15, P5 CONN15, P6 CONN15, P7 CONN15, P8 CONN15, P9 CONN15, Q2 MOSFET_NCHAN

Commit message: double checking, adding BOM
Parts:
- P1, P10, P11, P12, P2, P3, P4, P5, P6, P7, P8, P9: LCSC PN (none) -> C5210739; PN (none) -> PPPC151LFBN-RC
- Q2: LCSC PN (none) -> C165220; PN (none) -> ME2306D
- R1: LCSC PN (none) -> C17540; PN (none) -> 0805W8F2000T5E
- R2: LCSC PN (none) -> C4328; PN (none) -> 0805W8F2002T5E
Other:
- company: (none) -> IORodeo for Reiserlab @ Janelia
- title: (none) -> 12-12 NI G4.1 Arena Modular LED Display

Commit message: ready order ni and teensy 12-12, cleanup development
Other:
- note added: "ME2306D LCSC C165220"
- note removed: "SI2302-TP Digikey SI2302-TPMSCT-ND LCSC C4748714"
Changed lines of the file:
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@@
 		)
 	)
-	(text "SI2302-TP \nDigikey SI2302-TPMSCT-ND\nLCSC C4748714  \n"
+	(text "ME2306D\nLCSC C165220\n"
 		(exclude_from_sim no)
-		(at 63.5 121.92 0)
+		(at 66.04 117.348 0)
 		(effects
 			(font
@@
 					(size 1.524 1.524)
 				)
+				(hide yes)
 			)
 		)
