File: development/arena_12-12_w_vreg/teensy4p1/teensy_arena_12-12_v0p2/holes.kicad_sch (KiCad schematic)
At the start: 4 parts

Commit message: ready order ni and teensy 12-12, cleanup development
Parts:
- H1, H2, H3, H4: now not fitted
Other:
- company: (none) -> IORodeo for Reiserlab @ Janelia
- title: (none) -> 12-12 Teensy G4.1 Arena Modular LED Display
