File: development/arena_12-12_w_vreg/teensy4p1/teensy_arena_12-12_v0p2/level_shifters.kicad_sch (KiCad schematic)
At the start: 15 parts, among them U1 TXB0108PW, U2 TXB0108PW, U3 TXB0108PW, U4 TXB0108PW, U5 TXB0108PW

Commit message: ready order ni and teensy 12-12, cleanup development
Parts:
- C1, C10, C2, C3, C4, C5, C6, C7, C8, C9: DigiKey PN (none) -> 1276-1000-2-ND; LCSC PN (none) -> C1591; MPN (none) -> CL10B104KB8NNNC
- U1, U2, U3, U4, U5: DigiKey PN (none) -> 296-21527-2-ND; LCSC PN (none) -> C53406; MPN (none) -> TXB0108PWR
Other:
- company: (none) -> IORodeo for Reiserlab @ Janelia
- title: (none) -> 12-12 Teensy G4.1 Arena Modular LED Display
