File: development/arena_12-12_w_vreg/teensy4p1/teensy_arena_12-12_v0p2/panel_headers.kicad_sch (KiCad schematic)
At the start: 15 parts, among them P1 CONN15, P10 CONN15, P11 CONN15, P12 CONN15, P2 CONN15, P3 CONN15, P4 CONN15, P5 CONN15, P6 CONN15, P7 CONN15, P8 CONN15, P9 CONN15, Q2 MOSFET_NCHAN

Commit message: ready order ni and teensy 12-12, cleanup development
Parts:
- P1, P10, P11, P12, P2, P3, P4, P5, P6, P7, P8, P9: DigiKey PN (none) -> S7048-ND; LCSC PN (none) -> C5210739; MPN (none) -> PPPC151LFBN-RC
- Q2: LCSC PN (none) -> C165220; MPN (none) -> ME2306D
- R1: LCSC PN (none) -> C17540; MPN (none) -> 0805W8F2000T5E
- R2: LCSC PN (none) -> C4328; MPN (none) -> 0805W8F2002T5E
Other:
- note added: "ME2306D LCSC C165220"
- note removed: "Notes: Error on P2 and P2. PAN5V.CS_06 was repeated twice and PAN5V.CS_07 was missing."
- note removed: "SI2302-TP Digikey SI2302-TPMSCT-ND LCSC C4748714"
- company: (none) -> IORodeo for Reiserlab @ Janelia
- title: (none) -> 12-12 Teensy G4.1 Arena Modular LED Display
