File: development/arena_12-12_w_vreg/teensy4p1/teensy_arena_12-12_v0p2/power.kicad_sch (KiCad schematic)
At the start: 86 parts, among them J1 Barrel_Jack, SW1 SW_SPDT, U10 TPS564201DDC, U11 TPS564201DDC, U12 TPS564201DDC, U13 TPS564201DDC, U14 TPS564201DDC, U15 TPS564201DDC, U16 TPS564201DDC, U17 TPS564201DDC, U6 TPS564201DDC, U7 TPS564201DDC, U8 TPS564201DDC, U9 TPS564201DDC

Commit message: ready order ni and teensy 12-12, cleanup development
Parts:
- C11, C14, C17, C20, C23, C26, C29, C32, C35, C38, C41, C44: DigiKey PN (none) -> 1276-1869-2-ND; LCSC PN (none) -> C96446; MPN (none) -> CL10A106MA8NRNC
- C12, C15, C18, C21, C24, C27, C30, C33, C36, C39, C42, C45: DigiKey PN (none) -> 1276-1000-2-ND; LCSC PN (none) -> C1591; MPN (none) -> CL10B104KB8NNNC
- C13, C16, C19, C22, C25, C28, C31, C34, C37, C40, C43, C46: DigiKey PN (none) -> 1276-7076-2-ND; LCSC PN (none) -> C2762594; MPN (none) -> CL10A226MO7JZNC
- J1: DigiKey PN (none) -> CP-063AH-ND; LCSC PN (none) -> C2928097; MPN (none) -> PJ-063AH
- L1, L10, L11, L12, L2, L3, L4, L5, L6, L7, L8, L9: LCSC PN (none) -> C5189747; MPN (none) -> CYA0630-3.3UH
- R10, R12, R14, R16, R18, R20, R22, R24, R26, R4, R6, R8: DigiKey PN (none) -> YAG1236TR-ND; LCSC PN (none) -> C95204; MPN (none) -> RT0603BRD0710KL
- R11, R13, R15, R17, R19, R21, R23, R25, R3, R5, R7, R9: DigiKey PN (none) -> YAG4575TR-ND; LCSC PN (none) -> C705784; MPN (none) -> RT0603BRD0756K2L
- SW1: DigiKey PN (none) -> CKC5102-ND; LCSC PN (none) -> C2798743; MPN (none) -> L102021ML04Q
- U10, U11, U12, U13, U14, U15, U16, U17, U6, U7, U8, U9: DigiKey PN (none) -> 296-47373-2-ND; LCSC PN (none) -> C464812; MPN (none) -> TPS564201DDCR
Other:
- company: (none) -> IORodeo for Reiserlab @ Janelia
- title: (none) -> 12-12 Teensy G4.1 Arena Modular LED Display
