File: development/arena_12-12_w_vreg/teensy4p1/teensy_arena_12-12_v0p2/teensy.kicad_sch (KiCad schematic)
At the start: 3 parts, among them J2 Conn_01x04, J3 Conn_01x04, U18 Teensy4.1

Commit message: ready order ni and teensy 12-12, cleanup development
Parts:
- J2, J3: LCSC PN (none) -> C145956; MPN (none) -> 1.0T-4P
- U18: now not fitted
Other:
- company: (none) -> IORodeo for Reiserlab @ Janelia
- title: (none) -> 12-12 Teensy G4.1 Arena Modular LED Display
