File: development/arena_12-12_w_vreg/teensy4p1/teensy_arena_12-12_v0p2/teensy_arena_12-12.kicad_sch (KiCad schematic)
At the start: 0 parts

Commit message: ready order ni and teensy 12-12, cleanup development
Other:
- company: (none) -> IORodeo for Reiserlab @ Janelia
- title: (none) -> 12-12 Teensy G4.1 Arena Modular LED Display
