File: development/arena_12-12/teensy4p1/teensy_arena_12-12_v0p1/layout_tool/teensy_arena_12-12.kicad_pcb (KiCad board)
At the start: 4 copper layers, 51 parts, among them J1 Barrel_Jack, J2 Conn_01x04, J3 Conn_01x04, P1 CONN15, P10 CONN15, P11 CONN15, P12 CONN15, P2 CONN15, P3 CONN15, P4 CONN15, P5 CONN15, P6 CONN15, P7 CONN15, P8 CONN15, P9 CONN15, Q2 MOSFET_NCHAN, SW1 SW_SPDT, U1 TXB0108PW, U18 Teensy4.1, U2 TXB0108PW, U3 TXB0108PW, U4 TXB0108PW, U5 TXB0108PW

Commit message: Worked on 12-12 arena layout.
Parts:
- removed Q2: MOSFET_NCHAN, Package_TO_SOT_SMD:SOT-23-3
- removed the U1 at (280.9, 222.8)
- added C11: 0.1uF, Capacitor_SMD:C_0603_1608Metric, F.Cu at (-71.9, 138.1)
- added C12: 0.1uF, Capacitor_SMD:C_0603_1608Metric, F.Cu at (-71.9, 140.6)
- added C13: 0.1uF, Capacitor_SMD:C_0603_1608Metric, F.Cu at (-71.9, 143.1)
- added C14: 0.1uF, Capacitor_SMD:C_0603_1608Metric, F.Cu at (-71.9, 145.6)
- added C15: 0.1uF, Capacitor_SMD:C_0603_1608Metric, F.Cu at (-71.9, 148.1)
- added C16: 0.1uF, Capacitor_SMD:C_0603_1608Metric, F.Cu at (-71.9, 150.6)
- added C17: 0.1uF, Capacitor_SMD:C_0603_1608Metric, F.Cu at (-67.9, 115.5)
- added C18: 0.1uF, Capacitor_SMD:C_0603_1608Metric, F.Cu at (-67.9, 118.0)
- added C19: 0.1uF, Capacitor_SMD:C_0603_1608Metric, F.Cu at (-67.9, 120.5)
- added C20: 0.1uF, Capacitor_SMD:C_0603_1608Metric, F.Cu at (-67.9, 123.0)
- added C21: 0.1uF, Capacitor_SMD:C_0603_1608Metric, F.Cu at (-67.9, 125.5)
- added C22: 0.1uF, Capacitor_SMD:C_0603_1608Metric, F.Cu at (-67.9, 128.0)
- added C23: 0.1uF, Capacitor_SMD:C_0603_1608Metric, F.Cu at (-67.9, 130.5)
- added C24: 0.1uF, Capacitor_SMD:C_0603_1608Metric, F.Cu at (-67.9, 133.1)
- added C25: 0.1uF, Capacitor_SMD:C_0603_1608Metric, F.Cu at (-67.9, 135.6)
- added C26: 0.1uF, Capacitor_SMD:C_0603_1608Metric, F.Cu at (-67.9, 138.1)
- added C27: 0.1uF, Capacitor_SMD:C_0603_1608Metric, F.Cu at (-67.9, 140.6)
- added C28: 0.1uF, Capacitor_SMD:C_0603_1608Metric, F.Cu at (-67.9, 143.1)
- added C29: 0.1uF, Capacitor_SMD:C_0603_1608Metric, F.Cu at (-67.9, 145.6)
- added C30: 0.1uF, Capacitor_SMD:C_0603_1608Metric, F.Cu at (-67.9, 148.1)
- added C31: 0.1uF, Capacitor_SMD:C_0603_1608Metric, F.Cu at (-67.9, 150.6)
- added C32: 0.1uF, Capacitor_SMD:C_0603_1608Metric, F.Cu at (-63.8, 115.5)
- added C33: 0.1uF, Capacitor_SMD:C_0603_1608Metric, F.Cu at (-63.8, 118.0)
- added C34: 0.1uF, Capacitor_SMD:C_0603_1608Metric, F.Cu at (-63.8, 120.5)
- added C35: 0.1uF, Capacitor_SMD:C_0603_1608Metric, F.Cu at (-63.8, 123.0)
- added C36: 0.1uF, Capacitor_SMD:C_0603_1608Metric, F.Cu at (-63.8, 125.5)
- added C37: 0.1uF, Capacitor_SMD:C_0603_1608Metric, F.Cu at (-63.8, 128.0)
- added C38: 0.1uF, Capacitor_SMD:C_0603_1608Metric, F.Cu at (-63.8, 130.5)
- added C39: 0.1uF, Capacitor_SMD:C_0603_1608Metric, F.Cu at (-63.8, 133.1)
- added C40: 0.1uF, Capacitor_SMD:C_0603_1608Metric, F.Cu at (-63.8, 135.6)
- added C41: 0.1uF, Capacitor_SMD:C_0603_1608Metric, F.Cu at (-63.8, 138.1)
- added C42: 0.1uF, Capacitor_SMD:C_0603_1608Metric, F.Cu at (-63.8, 140.6)
- added C43: 0.1uF, Capacitor_SMD:C_0603_1608Metric, F.Cu at (-63.8, 143.1)
- added C44: 0.1uF, Capacitor_SMD:C_0603_1608Metric, F.Cu at (-63.8, 145.6)
- added C45: 0.1uF, Capacitor_SMD:C_0603_1608Metric, F.Cu at (-63.8, 148.1)
- added C46: 0.1uF, Capacitor_SMD:C_0603_1608Metric, F.Cu at (-63.8, 150.6)
- added C47: 0.1uF, Capacitor_SMD:C_0603_1608Metric, F.Cu at (272.5, 169.0)
- added C48: 0.1uF, Capacitor_SMD:C_0603_1608Metric, F.Cu at (272.4, 176.3)
- added C49: 0.1uF, Capacitor_SMD:C_0603_1608Metric, F.Cu at (272.4, 181.6)
- added C50: 0.1uF, Capacitor_SMD:C_0603_1608Metric, F.Cu at (272.5, 187.0)
- added C51: 0.1uF, Capacitor_SMD:C_0603_1608Metric, F.Cu at (-71.9, 80.9)
- added C52: 0.1uF, Capacitor_SMD:C_0603_1608Metric, F.Cu at (-71.9, 83.4)
- added C53: 0.1uF, Capacitor_SMD:C_0603_1608Metric, F.Cu at (-71.9, 85.9)
- added C54: 0.1uF, Capacitor_SMD:C_0603_1608Metric, F.Cu at (-71.9, 88.4)
- added C55: 0.1uF, Capacitor_SMD:C_0603_1608Metric, F.Cu at (-71.9, 90.9)
- added C56: 0.1uF, Capacitor_SMD:C_0603_1608Metric, F.Cu at (-71.9, 93.4)
- added C57: 0.1uF, Capacitor_SMD:C_0603_1608Metric, F.Cu at (-71.9, 95.9)
- added C58: 0.1uF, Capacitor_SMD:C_0603_1608Metric, F.Cu at (-71.9, 98.4)
- added C59: 0.1uF, Capacitor_SMD:C_0603_1608Metric, F.Cu at (-71.9, 100.9)
- added C60: 0.1uF, Capacitor_SMD:C_0603_1608Metric, F.Cu at (-71.9, 103.4)
- added C61: 0.1uF, Capacitor_SMD:C_0603_1608Metric, F.Cu at (-71.9, 106.0)
- added C62: 0.1uF, Capacitor_SMD:C_0603_1608Metric, F.Cu at (-71.9, 108.5)
- added C63: 0.1uF, Capacitor_SMD:C_0603_1608Metric, F.Cu at (-71.9, 111.0)
- added C64: 0.1uF, Capacitor_SMD:C_0603_1608Metric, F.Cu at (-67.9, 70.8)
- added C65: 0.1uF, Capacitor_SMD:C_0603_1608Metric, F.Cu at (-67.9, 73.3)
- added C66: 0.1uF, Capacitor_SMD:C_0603_1608Metric, F.Cu at (-67.9, 75.8)
- added C67: 0.1uF, Capacitor_SMD:C_0603_1608Metric, F.Cu at (-67.9, 78.3)
- added C68: 0.1uF, Capacitor_SMD:C_0603_1608Metric, F.Cu at (-67.9, 80.9)
- added C69: 0.1uF, Capacitor_SMD:C_0603_1608Metric, F.Cu at (-67.9, 83.4)
- added C70: 0.1uF, Capacitor_SMD:C_0603_1608Metric, F.Cu at (-67.9, 85.9)
- added C71: 0.1uF, Capacitor_SMD:C_0603_1608Metric, F.Cu at (-67.9, 88.4)
- added C72: 0.1uF, Capacitor_SMD:C_0603_1608Metric, F.Cu at (-67.9, 90.9)
- added C73: 0.1uF, Capacitor_SMD:C_0603_1608Metric, F.Cu at (-67.9, 93.4)
- added C74: 0.1uF, Capacitor_SMD:C_0603_1608Metric, F.Cu at (-67.9, 95.9)
- added C75: 0.1uF, Capacitor_SMD:C_0603_1608Metric, F.Cu at (-67.9, 98.4)
- added C76: 0.1uF, Capacitor_SMD:C_0603_1608Metric, F.Cu at (-67.9, 100.9)
- added C77: 0.1uF, Capacitor_SMD:C_0603_1608Metric, F.Cu at (-67.9, 103.4)
- added C78: 0.1uF, Capacitor_SMD:C_0603_1608Metric, F.Cu at (-67.9, 106.0)
- added C79: 0.1uF, Capacitor_SMD:C_0603_1608Metric, F.Cu at (-67.9, 108.5)
- added C80: 0.1uF, Capacitor_SMD:C_0603_1608Metric, F.Cu at (-67.9, 111.0)
- added C81: 0.1uF, Capacitor_SMD:C_0603_1608Metric, F.Cu at (-63.8, 70.8)
- added C82: 0.1uF, Capacitor_SMD:C_0603_1608Metric, F.Cu at (-63.8, 73.3)
- added C83: 0.1uF, Capacitor_SMD:C_0603_1608Metric, F.Cu at (-63.8, 75.8)
- added C84: 0.1uF, Capacitor_SMD:C_0603_1608Metric, F.Cu at (-63.8, 78.3)
- added C85: 0.1uF, Capacitor_SMD:C_0603_1608Metric, F.Cu at (-63.8, 80.9)
- added C86: 0.1uF, Capacitor_SMD:C_0603_1608Metric, F.Cu at (-63.8, 83.4)
- added C87: 0.1uF, Capacitor_SMD:C_0603_1608Metric, F.Cu at (-63.8, 85.9)
- added C88: 0.1uF, Capacitor_SMD:C_0603_1608Metric, F.Cu at (-63.8, 88.4)
- added C89: 0.1uF, Capacitor_SMD:C_0603_1608Metric, F.Cu at (-63.8, 90.9)
- added C90: 0.1uF, Capacitor_SMD:C_0603_1608Metric, F.Cu at (-63.8, 93.4)
- added C91: 0.1uF, Capacitor_SMD:C_0603_1608Metric, F.Cu at (-63.8, 95.9)
- added C92: 0.1uF, Capacitor_SMD:C_0603_1608Metric, F.Cu at (-63.8, 98.4)
- added C93: 0.1uF, Capacitor_SMD:C_0603_1608Metric, F.Cu at (-63.8, 100.9)
- added C94: 0.1uF, Capacitor_SMD:C_0603_1608Metric, F.Cu at (-63.8, 103.4)
- added J4: Barrel_Jack, arena_custom:DCJACK_2PIN_HIGHCURRENT, F.Cu at (95.0, 63.5)
- added Q1: MOSFET_NCHAN, Package_TO_SOT_SMD:SOT-23-3, F.Cu at (284.4, 130.8)
- added R10: 68, Resistor_SMD:R_0603_1608Metric, F.Cu at (275.6, 253.6)
- added R100: 68, Resistor_SMD:R_0603_1608Metric, F.Cu at (-43.8, 118.0)
- added R101: 68, Resistor_SMD:R_0603_1608Metric, F.Cu at (-43.8, 120.5)
- added R102: 68, Resistor_SMD:R_0603_1608Metric, F.Cu at (-43.8, 123.0)
- added R103: 68, Resistor_SMD:R_0603_1608Metric, F.Cu at (-43.8, 125.5)
- added R104: 68, Resistor_SMD:R_0603_1608Metric, F.Cu at (-43.8, 128.0)
- added R105: 68, Resistor_SMD:R_0603_1608Metric, F.Cu at (-43.8, 130.5)
- added R106: 68, Resistor_SMD:R_0603_1608Metric, F.Cu at (-43.8, 133.1)
- added R107: 68, Resistor_SMD:R_0603_1608Metric, F.Cu at (-43.8, 135.6)
- added R108: 68, Resistor_SMD:R_0603_1608Metric, F.Cu at (-43.8, 138.1)
- added R109: 68, Resistor_SMD:R_0603_1608Metric, F.Cu at (-43.8, 140.6)
- added R11: 68, Resistor_SMD:R_0603_1608Metric, F.Cu at (273.2, 254.3)
- added R110: 68, Resistor_SMD:R_0603_1608Metric, F.Cu at (-43.8, 143.1)
- added R111: 68, Resistor_SMD:R_0603_1608Metric, F.Cu at (-43.8, 145.6)
- added R112: 68, Resistor_SMD:R_0603_1608Metric, F.Cu at (-43.8, 148.1)
- added R113: 68, Resistor_SMD:R_0603_1608Metric, F.Cu at (-43.8, 150.6)
- added R114: 68, Resistor_SMD:R_0603_1608Metric, F.Cu at (-39.8, 115.5)
- added R115: 68, Resistor_SMD:R_0603_1608Metric, F.Cu at (-39.8, 118.0)
- added R116: 68, Resistor_SMD:R_0603_1608Metric, F.Cu at (-39.8, 120.5)
- added R117: 68, Resistor_SMD:R_0603_1608Metric, F.Cu at (-39.8, 123.0)
- added R118: 68, Resistor_SMD:R_0603_1608Metric, F.Cu at (-39.8, 125.5)
- added R119: 68, Resistor_SMD:R_0603_1608Metric, F.Cu at (-39.8, 128.0)
- added R12: 68, Resistor_SMD:R_0603_1608Metric, F.Cu at (-9.16, 120.5)
- added R120: 68, Resistor_SMD:R_0603_1608Metric, F.Cu at (-39.8, 130.5)
- added R121: 68, Resistor_SMD:R_0603_1608Metric, F.Cu at (-39.8, 133.1)
- added R122: 68, Resistor_SMD:R_0603_1608Metric, F.Cu at (-39.8, 135.6)
- added R123: 68, Resistor_SMD:R_0603_1608Metric, F.Cu at (-39.8, 138.1)
- added R124: 68, Resistor_SMD:R_0603_1608Metric, F.Cu at (-39.8, 140.6)
- added R125: 68, Resistor_SMD:R_0603_1608Metric, F.Cu at (-39.8, 143.1)
- added R126: 68, Resistor_SMD:R_0603_1608Metric, F.Cu at (-39.8, 145.6)
- added R127: 68, Resistor_SMD:R_0603_1608Metric, F.Cu at (272.5, 167.4)
- added R128: 68, Resistor_SMD:R_0603_1608Metric, F.Cu at (272.5, 170.6)
- added R129: 68, Resistor_SMD:R_0603_1608Metric, F.Cu at (272.5, 174.7)
- added R13: 68, Resistor_SMD:R_0603_1608Metric, F.Cu at (-9.16, 123.0)
- added R130: 68, Resistor_SMD:R_0603_1608Metric, F.Cu at (272.5, 178.0)
- added R131: 68, Resistor_SMD:R_0603_1608Metric, F.Cu at (272.4, 180.0)
- added R132: 68, Resistor_SMD:R_0603_1608Metric, F.Cu at (272.5, 183.4)
- added R133: 68, Resistor_SMD:R_0603_1608Metric, F.Cu at (272.5, 185.4)
- added R134: 68, Resistor_SMD:R_0603_1608Metric, F.Cu at (272.5, 188.7)
- added R135: 68, Resistor_SMD:R_0603_1608Metric, F.Cu at (-59.8, 83.4)
- added R136: 68, Resistor_SMD:R_0603_1608Metric, F.Cu at (-59.8, 85.9)
- added R137: 68, Resistor_SMD:R_0603_1608Metric, F.Cu at (-59.8, 88.4)
- added R138: 68, Resistor_SMD:R_0603_1608Metric, F.Cu at (-59.8, 90.9)
- added R139: 68, Resistor_SMD:R_0603_1608Metric, F.Cu at (-59.8, 93.4)
- added R14: 68, Resistor_SMD:R_0603_1608Metric, F.Cu at (-9.16, 125.5)
- added R140: 68, Resistor_SMD:R_0603_1608Metric, F.Cu at (-59.8, 95.9)
- added R141: 68, Resistor_SMD:R_0603_1608Metric, F.Cu at (-59.8, 98.4)
- added R142: 68, Resistor_SMD:R_0603_1608Metric, F.Cu at (-59.8, 100.9)
- added R143: 68, Resistor_SMD:R_0603_1608Metric, F.Cu at (-59.8, 103.4)
- added R144: 68, Resistor_SMD:R_0603_1608Metric, F.Cu at (-59.8, 106.0)
- added R145: 68, Resistor_SMD:R_0603_1608Metric, F.Cu at (-59.8, 108.5)
- added R146: 68, Resistor_SMD:R_0603_1608Metric, F.Cu at (-59.8, 111.0)
- added R147: 68, Resistor_SMD:R_0603_1608Metric, F.Cu at (-55.8, 70.8)
- added R148: 68, Resistor_SMD:R_0603_1608Metric, F.Cu at (-55.8, 73.3)
- added R149: 68, Resistor_SMD:R_0603_1608Metric, F.Cu at (-55.8, 75.8)
- added R15: 68, Resistor_SMD:R_0603_1608Metric, F.Cu at (-9.16, 128.0)
- added R150: 68, Resistor_SMD:R_0603_1608Metric, F.Cu at (-55.8, 78.3)
- added R151: 68, Resistor_SMD:R_0603_1608Metric, F.Cu at (-55.8, 80.9)
- added R152: 68, Resistor_SMD:R_0603_1608Metric, F.Cu at (-55.8, 83.4)
- added R153: 68, Resistor_SMD:R_0603_1608Metric, F.Cu at (-55.8, 85.9)
- added R154: 68, Resistor_SMD:R_0603_1608Metric, F.Cu at (-55.8, 88.4)
- added R155: 68, Resistor_SMD:R_0603_1608Metric, F.Cu at (-55.8, 90.9)
- added R156: 68, Resistor_SMD:R_0603_1608Metric, F.Cu at (-55.8, 93.4)
- added R157: 68, Resistor_SMD:R_0603_1608Metric, F.Cu at (-55.8, 95.9)
- added R158: 68, Resistor_SMD:R_0603_1608Metric, F.Cu at (-55.8, 98.4)
- added R159: 68, Resistor_SMD:R_0603_1608Metric, F.Cu at (-55.8, 100.9)
- added R16: 68, Resistor_SMD:R_0603_1608Metric, F.Cu at (-9.16, 130.5)
- added R160: 68, Resistor_SMD:R_0603_1608Metric, F.Cu at (-55.8, 103.4)
- added R161: 68, Resistor_SMD:R_0603_1608Metric, F.Cu at (-55.8, 106.0)
- added R162: 68, Resistor_SMD:R_0603_1608Metric, F.Cu at (-55.8, 108.5)
- added R163: 68, Resistor_SMD:R_0603_1608Metric, F.Cu at (-55.8, 111.0)
- added R164: 68, Resistor_SMD:R_0603_1608Metric, F.Cu at (-51.8, 70.8)
- added R165: 68, Resistor_SMD:R_0603_1608Metric, F.Cu at (-51.8, 73.3)
- added R166: 68, Resistor_SMD:R_0603_1608Metric, F.Cu at (-51.8, 75.8)
- added R167: 68, Resistor_SMD:R_0603_1608Metric, F.Cu at (-51.8, 78.3)
- added R168: 68, Resistor_SMD:R_0603_1608Metric, F.Cu at (-51.8, 80.9)
- added R169: 68, Resistor_SMD:R_0603_1608Metric, F.Cu at (-51.8, 83.4)
- added R17: 68, Resistor_SMD:R_0603_1608Metric, F.Cu at (-9.16, 133.1)
- added R170: 68, Resistor_SMD:R_0603_1608Metric, F.Cu at (-51.8, 85.9)
- added R171: 68, Resistor_SMD:R_0603_1608Metric, F.Cu at (-51.8, 88.4)
- added R172: 68, Resistor_SMD:R_0603_1608Metric, F.Cu at (-51.8, 90.9)
- added R173: 68, Resistor_SMD:R_0603_1608Metric, F.Cu at (-51.8, 93.4)
- added R174: 68, Resistor_SMD:R_0603_1608Metric, F.Cu at (-51.8, 95.9)
- added R175: 68, Resistor_SMD:R_0603_1608Metric, F.Cu at (-51.8, 98.4)
- added R176: 68, Resistor_SMD:R_0603_1608Metric, F.Cu at (-51.8, 100.9)
- added R177: 68, Resistor_SMD:R_0603_1608Metric, F.Cu at (-51.8, 103.4)
- added R178: 68, Resistor_SMD:R_0603_1608Metric, F.Cu at (-51.8, 106.0)
- added R179: 68, Resistor_SMD:R_0603_1608Metric, F.Cu at (-51.8, 108.5)
- added R18: 68, Resistor_SMD:R_0603_1608Metric, F.Cu at (-5.15, 115.5)
- added R180: 68, Resistor_SMD:R_0603_1608Metric, F.Cu at (-51.8, 111.0)
- added R181: 68, Resistor_SMD:R_0603_1608Metric, F.Cu at (-47.8, 70.8)
- added R182: 68, Resistor_SMD:R_0603_1608Metric, F.Cu at (-47.8, 73.3)
- added R183: 68, Resistor_SMD:R_0603_1608Metric, F.Cu at (-47.8, 75.8)
- added R184: 68, Resistor_SMD:R_0603_1608Metric, F.Cu at (-47.8, 78.3)
- added R185: 68, Resistor_SMD:R_0603_1608Metric, F.Cu at (-47.8, 80.9)
- added R186: 68, Resistor_SMD:R_0603_1608Metric, F.Cu at (-47.8, 83.4)
- added R187: 68, Resistor_SMD:R_0603_1608Metric, F.Cu at (-47.8, 85.9)
- added R188: 68, Resistor_SMD:R_0603_1608Metric, F.Cu at (-47.8, 88.4)
- added R189: 68, Resistor_SMD:R_0603_1608Metric, F.Cu at (-47.8, 90.9)
- added R19: 68, Resistor_SMD:R_0603_1608Metric, F.Cu at (-5.15, 118.0)
- added R190: 68, Resistor_SMD:R_0603_1608Metric, F.Cu at (-47.8, 93.4)
- added R191: 68, Resistor_SMD:R_0603_1608Metric, F.Cu at (-47.8, 95.9)
- added R192: 68, Resistor_SMD:R_0603_1608Metric, F.Cu at (-47.8, 98.4)
- added R193: 68, Resistor_SMD:R_0603_1608Metric, F.Cu at (-47.8, 100.9)
- added R194: 68, Resistor_SMD:R_0603_1608Metric, F.Cu at (-47.8, 103.4)
- added R195: 68, Resistor_SMD:R_0603_1608Metric, F.Cu at (-47.8, 106.0)
- added R196: 68, Resistor_SMD:R_0603_1608Metric, F.Cu at (-47.8, 108.5)
- added R197: 68, Resistor_SMD:R_0603_1608Metric, F.Cu at (-47.8, 111.0)
- added R198: 68, Resistor_SMD:R_0603_1608Metric, F.Cu at (-43.8, 70.8)
- added R199: 68, Resistor_SMD:R_0603_1608Metric, F.Cu at (-43.8, 73.3)
- added R20: 68, Resistor_SMD:R_0603_1608Metric, F.Cu at (-5.15, 120.5)
- added R200: 68, Resistor_SMD:R_0603_1608Metric, F.Cu at (-43.8, 75.8)
- added R201: 68, Resistor_SMD:R_0603_1608Metric, F.Cu at (-43.8, 78.3)
- added R202: 68, Resistor_SMD:R_0603_1608Metric, F.Cu at (-43.8, 80.9)
- added R203: 68, Resistor_SMD:R_0603_1608Metric, F.Cu at (-43.8, 83.4)
- added R204: 68, Resistor_SMD:R_0603_1608Metric, F.Cu at (-43.8, 85.9)
- added R205: 68, Resistor_SMD:R_0603_1608Metric, F.Cu at (-43.8, 88.4)
- added R206: 68, Resistor_SMD:R_0603_1608Metric, F.Cu at (-43.8, 90.9)
- added R207: 68, Resistor_SMD:R_0603_1608Metric, F.Cu at (-43.8, 93.4)
- added R208: 68, Resistor_SMD:R_0603_1608Metric, F.Cu at (-43.8, 95.9)
- added R209: 68, Resistor_SMD:R_0603_1608Metric, F.Cu at (-43.8, 98.4)
- added R21: 68, Resistor_SMD:R_0603_1608Metric, F.Cu at (-5.15, 123.0)
- added R210: 68, Resistor_SMD:R_0603_1608Metric, F.Cu at (-43.8, 100.9)
- added R211: 68, Resistor_SMD:R_0603_1608Metric, F.Cu at (-43.8, 103.4)
- added R212: 68, Resistor_SMD:R_0603_1608Metric, F.Cu at (-43.8, 106.0)
- added R213: 68, Resistor_SMD:R_0603_1608Metric, F.Cu at (-43.8, 108.5)
- added R214: 68, Resistor_SMD:R_0603_1608Metric, F.Cu at (-43.8, 111.0)
- added R215: 68, Resistor_SMD:R_0603_1608Metric, F.Cu at (-39.8, 70.8)
- added R216: 68, Resistor_SMD:R_0603_1608Metric, F.Cu at (-39.8, 73.3)
- added R217: 68, Resistor_SMD:R_0603_1608Metric, F.Cu at (-39.8, 75.8)
- added R218: 68, Resistor_SMD:R_0603_1608Metric, F.Cu at (-39.8, 78.3)
- added R219: 68, Resistor_SMD:R_0603_1608Metric, F.Cu at (-39.8, 80.9)
- added R22: 68, Resistor_SMD:R_0603_1608Metric, F.Cu at (-5.15, 125.5)
- added R220: 68, Resistor_SMD:R_0603_1608Metric, F.Cu at (-39.8, 83.4)
- added R221: 68, Resistor_SMD:R_0603_1608Metric, F.Cu at (-39.8, 85.9)
- added R222: 68, Resistor_SMD:R_0603_1608Metric, F.Cu at (-39.8, 88.4)
- added R223: 68, Resistor_SMD:R_0603_1608Metric, F.Cu at (272.5, 172.7)
- added R224: 68, Resistor_SMD:R_0603_1608Metric, F.Cu at (-64.5, 187.8)
- added R225: 68, Resistor_SMD:R_0603_1608Metric, F.Cu at (-64.5, 190.3)
- added R226: 68, Resistor_SMD:R_0603_1608Metric, F.Cu at (-64.5, 192.8)
- added R227: 68, Resistor_SMD:R_0603_1608Metric, F.Cu at (-60.5, 185.3)
- added R228: 68, Resistor_SMD:R_0603_1608Metric, F.Cu at (-60.5, 187.8)
- added R229: 68, Resistor_SMD:R_0603_1608Metric, F.Cu at (-60.5, 190.3)
- added R23: 68, Resistor_SMD:R_0603_1608Metric, F.Cu at (-5.15, 128.0)
- added R230: 68, Resistor_SMD:R_0603_1608Metric, F.Cu at (-60.5, 192.8)
- added R231: 68, Resistor_SMD:R_0603_1608Metric, F.Cu at (-56.5, 185.3)
- added R232: 68, Resistor_SMD:R_0603_1608Metric, F.Cu at (-56.5, 187.8)
- added R233: 68, Resistor_SMD:R_0603_1608Metric, F.Cu at (-56.5, 190.3)
- added R234: 68, Resistor_SMD:R_0603_1608Metric, F.Cu at (-56.5, 192.8)
- added R24: 68, Resistor_SMD:R_0603_1608Metric, F.Cu at (-5.15, 130.5)
- added R25: 68, Resistor_SMD:R_0603_1608Metric, F.Cu at (-5.15, 133.1)
- added R26: 68, Resistor_SMD:R_0603_1608Metric, F.Cu at (-1.14, 115.5)
- added R27: 68, Resistor_SMD:R_0603_1608Metric, F.Cu at (-1.14, 118.0)
- added R28: 68, Resistor_SMD:R_0603_1608Metric, F.Cu at (-1.14, 120.5)
- added R29: 68, Resistor_SMD:R_0603_1608Metric, F.Cu at (-1.14, 123.0)
- added R3: 68, Resistor_SMD:R_0603_1608Metric, F.Cu at (-13.2, 118.0)
- added R30: 68, Resistor_SMD:R_0603_1608Metric, F.Cu at (-1.14, 125.5)
- added R31: 68, Resistor_SMD:R_0603_1608Metric, F.Cu at (-1.14, 128.0)
- added R32: 68, Resistor_SMD:R_0603_1608Metric, F.Cu at (-1.14, 130.5)
- added R33: 68, Resistor_SMD:R_0603_1608Metric, F.Cu at (-1.14, 133.1)
- added R34: 68, Resistor_SMD:R_0603_1608Metric, F.Cu at (2.87, 115.5)
- added R35: 68, Resistor_SMD:R_0603_1608Metric, F.Cu at (2.87, 118.0)
- added R36: 68, Resistor_SMD:R_0603_1608Metric, F.Cu at (2.87, 120.5)
- added R37: 68, Resistor_SMD:R_0603_1608Metric, F.Cu at (2.87, 123.0)
- added R38: 68, Resistor_SMD:R_0603_1608Metric, F.Cu at (2.87, 125.5)
- added R39: 68, Resistor_SMD:R_0603_1608Metric, F.Cu at (-59.8, 115.5)
- added R4: 68, Resistor_SMD:R_0603_1608Metric, F.Cu at (259.3, 276.0)
- added R40: 68, Resistor_SMD:R_0603_1608Metric, F.Cu at (-59.8, 118.0)
- added R41: 68, Resistor_SMD:R_0603_1608Metric, F.Cu at (-59.8, 120.5)
- added R42: 68, Resistor_SMD:R_0603_1608Metric, F.Cu at (-59.8, 123.0)
- added R43: 68, Resistor_SMD:R_0603_1608Metric, F.Cu at (-59.8, 125.5)
- added R44: 68, Resistor_SMD:R_0603_1608Metric, F.Cu at (-59.8, 128.0)
- added R45: 68, Resistor_SMD:R_0603_1608Metric, F.Cu at (-59.8, 130.5)
- added R46: 68, Resistor_SMD:R_0603_1608Metric, F.Cu at (-59.8, 133.1)
- added R47: 68, Resistor_SMD:R_0603_1608Metric, F.Cu at (-59.8, 135.6)
- added R48: 68, Resistor_SMD:R_0603_1608Metric, F.Cu at (-59.8, 138.1)
- added R49: 68, Resistor_SMD:R_0603_1608Metric, F.Cu at (-59.8, 140.6)
- added R5: 68, Resistor_SMD:R_0603_1608Metric, F.Cu at (256.5, 260.4)
- added R50: 68, Resistor_SMD:R_0603_1608Metric, F.Cu at (-59.8, 143.1)
- added R51: 68, Resistor_SMD:R_0603_1608Metric, F.Cu at (-59.8, 145.6)
- added R52: 68, Resistor_SMD:R_0603_1608Metric, F.Cu at (-59.8, 148.1)
- added R53: 68, Resistor_SMD:R_0603_1608Metric, F.Cu at (-59.8, 150.6)
- added R54: 68, Resistor_SMD:R_0603_1608Metric, F.Cu at (-55.8, 115.5)
- added R55: 68, Resistor_SMD:R_0603_1608Metric, F.Cu at (-55.8, 118.0)
- added R56: 68, Resistor_SMD:R_0603_1608Metric, F.Cu at (-55.8, 120.5)
- added R57: 68, Resistor_SMD:R_0603_1608Metric, F.Cu at (-55.8, 123.0)
- added R58: 68, Resistor_SMD:R_0603_1608Metric, F.Cu at (-55.8, 125.5)
- added R59: 68, Resistor_SMD:R_0603_1608Metric, F.Cu at (-55.8, 128.0)
- added R6: 68, Resistor_SMD:R_0603_1608Metric, F.Cu at (242.3, 265.4)
- added R60: 68, Resistor_SMD:R_0603_1608Metric, F.Cu at (-55.8, 130.5)
- added R61: 68, Resistor_SMD:R_0603_1608Metric, F.Cu at (-55.8, 133.1)
- added R62: 68, Resistor_SMD:R_0603_1608Metric, F.Cu at (-55.8, 135.6)
- added R63: 68, Resistor_SMD:R_0603_1608Metric, F.Cu at (-55.8, 138.1)
- added R64: 68, Resistor_SMD:R_0603_1608Metric, F.Cu at (-55.8, 140.6)
- added R65: 68, Resistor_SMD:R_0603_1608Metric, F.Cu at (-55.8, 143.1)
- added R66: 68, Resistor_SMD:R_0603_1608Metric, F.Cu at (-55.8, 145.6)
- added R67: 68, Resistor_SMD:R_0603_1608Metric, F.Cu at (-55.8, 148.1)
- added R68: 68, Resistor_SMD:R_0603_1608Metric, F.Cu at (-55.8, 150.6)
- added R69: 68, Resistor_SMD:R_0603_1608Metric, F.Cu at (-51.8, 115.5)
- added R7: 68, Resistor_SMD:R_0603_1608Metric, F.Cu at (244.6, 264.8)
- added R70: 68, Resistor_SMD:R_0603_1608Metric, F.Cu at (-51.8, 118.0)
- added R71: 68, Resistor_SMD:R_0603_1608Metric, F.Cu at (-51.8, 120.5)
- added R72: 68, Resistor_SMD:R_0603_1608Metric, F.Cu at (-51.8, 123.0)
- added R73: 68, Resistor_SMD:R_0603_1608Metric, F.Cu at (-51.8, 125.5)
- added R74: 68, Resistor_SMD:R_0603_1608Metric, F.Cu at (-51.8, 128.0)
- added R75: 68, Resistor_SMD:R_0603_1608Metric, F.Cu at (-51.8, 130.5)
- added R76: 68, Resistor_SMD:R_0603_1608Metric, F.Cu at (-51.8, 133.1)
- added R77: 68, Resistor_SMD:R_0603_1608Metric, F.Cu at (-51.8, 135.6)
- added R78: 68, Resistor_SMD:R_0603_1608Metric, F.Cu at (-51.8, 138.1)
- added R79: 68, Resistor_SMD:R_0603_1608Metric, F.Cu at (-51.8, 140.6)
- added R8: 68, Resistor_SMD:R_0603_1608Metric, F.Cu at (282.7, 251.0)
- added R80: 68, Resistor_SMD:R_0603_1608Metric, F.Cu at (-51.8, 143.1)
- added R81: 68, Resistor_SMD:R_0603_1608Metric, F.Cu at (-51.8, 145.6)
- added R82: 68, Resistor_SMD:R_0603_1608Metric, F.Cu at (-51.8, 148.1)
- added R83: 68, Resistor_SMD:R_0603_1608Metric, F.Cu at (-51.8, 150.6)
- added R84: 68, Resistor_SMD:R_0603_1608Metric, F.Cu at (-47.8, 115.5)
- added R85: 68, Resistor_SMD:R_0603_1608Metric, F.Cu at (-47.8, 118.0)
- added R86: 68, Resistor_SMD:R_0603_1608Metric, F.Cu at (-47.8, 120.5)
- added R87: 68, Resistor_SMD:R_0603_1608Metric, F.Cu at (-47.8, 123.0)
- added R88: 68, Resistor_SMD:R_0603_1608Metric, F.Cu at (-47.8, 125.5)
- added R89: 68, Resistor_SMD:R_0603_1608Metric, F.Cu at (-47.8, 128.0)
- added R9: 68, Resistor_SMD:R_0603_1608Metric, F.Cu at (277.9, 252.7)
- added R90: 68, Resistor_SMD:R_0603_1608Metric, F.Cu at (-47.8, 130.5)
- added R91: 68, Resistor_SMD:R_0603_1608Metric, F.Cu at (-47.8, 133.1)
- added R92: 68, Resistor_SMD:R_0603_1608Metric, F.Cu at (-47.8, 135.6)
- added R93: 68, Resistor_SMD:R_0603_1608Metric, F.Cu at (-47.8, 138.1)
- added R94: 68, Resistor_SMD:R_0603_1608Metric, F.Cu at (-47.8, 140.6)
- added R95: 68, Resistor_SMD:R_0603_1608Metric, F.Cu at (-47.8, 143.1)
- added R96: 68, Resistor_SMD:R_0603_1608Metric, F.Cu at (-47.8, 145.6)
- added R97: 68, Resistor_SMD:R_0603_1608Metric, F.Cu at (-47.8, 148.1)
- added R98: 68, Resistor_SMD:R_0603_1608Metric, F.Cu at (-47.8, 150.6)
- added R99: 68, Resistor_SMD:R_0603_1608Metric, F.Cu at (-43.8, 115.5)
- added U10: TXB0108PW, Package_SO:TSSOP-20_4.4x6.5mm_P0.65mm, F.Cu at (-52.0, 164.0)
- added U11: TXB0108PW, Package_SO:TSSOP-20_4.4x6.5mm_P0.65mm, F.Cu at (-52.0, 172.0)
- added U12: TXB0108PW, Package_SO:TSSOP-20_4.4x6.5mm_P0.65mm, F.Cu at (-43.2, 155.9)
- added U13: TXB0108PW, Package_SO:TSSOP-20_4.4x6.5mm_P0.65mm, F.Cu at (-43.2, 164.0)
- added U14: TXB0108PW, Package_SO:TSSOP-20_4.4x6.5mm_P0.65mm, F.Cu at (-43.2, 172.0)
- added U15: 74LVC1G17, Package_TO_SOT_SMD:SOT-23-5, F.Cu at (-35.2, 116.5)
- added U16: 74LVC1G17, Package_TO_SOT_SMD:SOT-23-5, F.Cu at (-35.2, 120.9)
- added U17: 74LVC1G17, Package_TO_SOT_SMD:SOT-23-5, F.Cu at (-35.2, 125.4)
- added U18: 74LVC1G17, Package_TO_SOT_SMD:SOT-23-5, F.Cu at (-35.2, 129.8)
- added U19: 74LVC2G17, Package_TO_SOT_SMD:SOT-23-6, F.Cu at (-35.2, 134.3)
- added U20: 74LVC2G17, Package_TO_SOT_SMD:SOT-23-6, F.Cu at (-35.2, 138.7)
- added U21: 74LVC2G17, Package_TO_SOT_SMD:SOT-23-6, F.Cu at (-30.1, 116.5)
- added U22: 74LVC2G17, Package_TO_SOT_SMD:SOT-23-6, F.Cu at (-30.1, 120.9)
- added U23: 74LVC2G17, Package_TO_SOT_SMD:SOT-23-6, F.Cu at (-30.1, 125.4)
- added U24: 74LVC2G17, Package_TO_SOT_SMD:SOT-23-6, F.Cu at (-30.1, 129.8)
- added U25: 74LVC2G17, Package_TO_SOT_SMD:SOT-23-6, F.Cu at (-30.1, 134.3)
- added U26: 74LVC2G17, Package_TO_SOT_SMD:SOT-23-6, F.Cu at (-30.1, 138.7)
- added U27: 74LVC2G17, Package_TO_SOT_SMD:SOT-23-6, F.Cu at (-24.9, 116.5)
- added U28: 74LVC2G17, Package_TO_SOT_SMD:SOT-23-6, F.Cu at (-24.9, 120.9)
- added U29: 74LVC2G17, Package_TO_SOT_SMD:SOT-23-6, F.Cu at (-24.9, 125.4)
- added U30: 74LVC2G17, Package_TO_SOT_SMD:SOT-23-6, F.Cu at (-24.9, 129.8)
- added U31: 74LVC2G17, Package_TO_SOT_SMD:SOT-23-6, F.Cu at (-24.9, 134.3)
- added U32: 74LVC2G17, Package_TO_SOT_SMD:SOT-23-6, F.Cu at (-24.9, 138.7)
- added U33: 74LVC2G17, Package_TO_SOT_SMD:SOT-23-6, F.Cu at (-19.8, 116.5)
- added U34: 74LVC2G17, Package_TO_SOT_SMD:SOT-23-6, F.Cu at (-19.8, 120.9)
- added U35: 74LVC2G17, Package_TO_SOT_SMD:SOT-23-6, F.Cu at (-19.8, 125.4)
- added U36: 74LVC2G17, Package_TO_SOT_SMD:SOT-23-6, F.Cu at (276.4, 169.0)
- added U37: 74LVC2G17, Package_TO_SOT_SMD:SOT-23-6, F.Cu at (276.4, 176.4)
- added U38: 74LVC2G17, Package_TO_SOT_SMD:SOT-23-6, F.Cu at (276.4, 181.6)
- added U39: 74LVC2G17, Package_TO_SOT_SMD:SOT-23-6, F.Cu at (276.4, 187.0)
- added U40: 74LVC2G17, Package_TO_SOT_SMD:SOT-23-6, F.Cu at (-35.2, 94.0)
- added U41: 74LVC2G17, Package_TO_SOT_SMD:SOT-23-6, F.Cu at (-35.2, 98.5)
- added U42: 74LVC2G17, Package_TO_SOT_SMD:SOT-23-6, F.Cu at (-30.1, 71.8)
- added U43: 74LVC2G17, Package_TO_SOT_SMD:SOT-23-6, F.Cu at (-30.1, 76.2)
- added U44: 74LVC2G17, Package_TO_SOT_SMD:SOT-23-6, F.Cu at (-30.1, 80.7)
- added U45: 74LVC2G17, Package_TO_SOT_SMD:SOT-23-6, F.Cu at (-30.1, 85.1)
- added U46: 74LVC2G17, Package_TO_SOT_SMD:SOT-23-6, F.Cu at (-30.1, 89.6)
- added U47: 74LVC2G17, Package_TO_SOT_SMD:SOT-23-6, F.Cu at (-30.1, 94.0)
- added U48: 74LVC2G17, Package_TO_SOT_SMD:SOT-23-6, F.Cu at (-30.1, 98.5)
- added U49: 74LVC2G17, Package_TO_SOT_SMD:SOT-23-6, F.Cu at (-24.9, 71.8)
- added U50: 74LVC2G17, Package_TO_SOT_SMD:SOT-23-6, F.Cu at (-24.9, 76.2)
- added U51: 74LVC2G17, Package_TO_SOT_SMD:SOT-23-6, F.Cu at (-24.9, 80.7)
- added U52: 74LVC2G17, Package_TO_SOT_SMD:SOT-23-6, F.Cu at (-24.9, 85.1)
- added U53: 74LVC2G17, Package_TO_SOT_SMD:SOT-23-6, F.Cu at (-24.9, 89.6)
- added U54: 74LVC2G17, Package_TO_SOT_SMD:SOT-23-6, F.Cu at (-24.9, 94.0)
- added U55: 74LVC2G17, Package_TO_SOT_SMD:SOT-23-6, F.Cu at (-24.9, 98.5)
- added U56: 74LVC2G17, Package_TO_SOT_SMD:SOT-23-6, F.Cu at (-19.8, 71.8)
- added U57: 74LVC2G17, Package_TO_SOT_SMD:SOT-23-6, F.Cu at (-19.8, 76.2)
- added U58: 74LVC2G17, Package_TO_SOT_SMD:SOT-23-6, F.Cu at (-19.8, 80.7)
- added U59: 74LVC2G17, Package_TO_SOT_SMD:SOT-23-6, F.Cu at (-19.8, 85.1)
- added U6: TXB0108PW, Package_SO:TSSOP-20_4.4x6.5mm_P0.65mm, F.Cu at (-60.7, 155.9)
- added U60: 74LVC2G17, Package_TO_SOT_SMD:SOT-23-6, F.Cu at (-19.8, 89.6)
- added U61: 74LVC2G17, Package_TO_SOT_SMD:SOT-23-6, F.Cu at (-19.8, 94.0)
- added U62: 74LVC2G17, Package_TO_SOT_SMD:SOT-23-6, F.Cu at (-19.8, 98.5)
- added U63: 74LVC2G17, Package_TO_SOT_SMD:SOT-23-6, F.Cu at (-14.6, 71.8)
- added U64: 74LVC2G17, Package_TO_SOT_SMD:SOT-23-6, F.Cu at (-14.6, 76.2)
- added U65: 74LVC2G17, Package_TO_SOT_SMD:SOT-23-6, F.Cu at (-14.6, 80.7)
- added U66: 74LVC2G17, Package_TO_SOT_SMD:SOT-23-6, F.Cu at (-14.6, 85.1)
- added U67: 74LVC2G17, Package_TO_SOT_SMD:SOT-23-6, F.Cu at (-14.6, 89.6)
- added U68: 74LVC2G17, Package_TO_SOT_SMD:SOT-23-6, F.Cu at (-14.6, 94.0)
- added U69: 74LVC2G17, Package_TO_SOT_SMD:SOT-23-6, F.Cu at (-14.6, 98.5)
- added U7: TXB0108PW, Package_SO:TSSOP-20_4.4x6.5mm_P0.65mm, F.Cu at (-60.7, 164.0)
- added U70: 74LVC2G17, Package_TO_SOT_SMD:SOT-23-6, F.Cu at (-9.45, 71.8)
- added U71: 74LVC2G17, Package_TO_SOT_SMD:SOT-23-6, F.Cu at (-9.45, 76.2)
- added U72: 74LVC2G17, Package_TO_SOT_SMD:SOT-23-6, F.Cu at (-9.45, 80.7)
- added U73: 74LVC2G17, Package_TO_SOT_SMD:SOT-23-6, F.Cu at (-9.45, 85.1)
- added U74: 74LVC2G17, Package_TO_SOT_SMD:SOT-23-6, F.Cu at (-9.45, 89.6)
- added U75: 74LVC2G17, Package_TO_SOT_SMD:SOT-23-6, F.Cu at (-9.45, 94.0)
- added U76: 74LVC2G17, Package_TO_SOT_SMD:SOT-23-6, F.Cu at (-9.45, 98.5)
- added U77: 74LVC2G17, Package_TO_SOT_SMD:SOT-23-6, F.Cu at (-4.30, 71.8)
- added U78: 74LVC2G17, Package_TO_SOT_SMD:SOT-23-6, F.Cu at (-4.30, 76.2)
- added U79: 74LVC2G17, Package_TO_SOT_SMD:SOT-23-6, F.Cu at (-4.30, 80.7)
- added U8: TXB0108PW, Package_SO:TSSOP-20_4.4x6.5mm_P0.65mm, F.Cu at (-60.7, 172.0)
- added U80: 74LVC2G17, Package_TO_SOT_SMD:SOT-23-6, F.Cu at (-4.30, 85.1)
- added U81: 74LVC2G17, Package_TO_SOT_SMD:SOT-23-6, F.Cu at (-4.30, 89.6)
- added U82: 74LVC2G17, Package_TO_SOT_SMD:SOT-23-6, F.Cu at (-4.30, 94.0)
- added U83: 74LVC2G17, Package_TO_SOT_SMD:SOT-23-6, F.Cu at (-4.30, 98.5)
- added U9: TXB0108PW, Package_SO:TSSOP-20_4.4x6.5mm_P0.65mm, F.Cu at (-52.0, 155.9)
- U2: value TXB0108PW -> 74LVC2G17; footprint Package_SO:TSSOP-20_4.4x6.5mm_P0.65mm -> Package_TO_SOT_SMD:SOT-23-6
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- renumbered C16 to C100, C17 to C101, C18 to C102, C19 to C103, C20 to C104, C21 to C105, C22 to C106, C11 to C95, C12 to C96, C13 to C97, C14 to C98, C15 to C99, U18 to U1
Connections:
- net /Panel Headers/RESET renamed /Panel Headers/HDR_RESET
- net Net-(SW1-A) renamed /Power/SW_5V
- C10 pad 1: +5V -> +3.3V
- C2 pad 1: +5V -> +3.3V
- C3 pad 1: +3.3V -> +5V
- C4 pad 1: +5V -> +3.3V
- C5 pad 1: +3.3V -> +5V
- C6 pad 1: +5V -> +3.3V
- C7 pad 1: +3.3V -> +5V
- C8 pad 1: +5V -> +3.3V
- C9 pad 1: +3.3V -> +5V
- P1 pad 10: /Level Shifters/PAN5V.CS_03 -> /Panel Headers/HDR_CS_03_P1
- P1 pad 11: /Level Shifters/PAN5V.CS_04 -> /Panel Headers/HDR_CS_04_P1
- P1 pad 15: /Level Shifters/PAN5V.EXT_INT -> /Panel Headers/HDR_EXT_INT_P1
- P1 pad 4: /Level Shifters/PAN5V.SCK_0 -> /Panel Headers/HDR_SCK_0_P1
- P1 pad 5: /Level Shifters/PAN5V.MOSI_0 -> /Panel Headers/HDR_MOSI_0_P1
- P1 pad 6: /Level Shifters/PAN5V.MISO_0 -> /Panel Headers/HDR_MISO_0_P1
- P1 pad 7: /Level Shifters/PAN5V.CS_00 -> /Panel Headers/HDR_CS_00_P1
- P1 pad 8: /Level Shifters/PAN5V.CS_01 -> /Panel Headers/HDR_CS_01_P1
- P1 pad 9: /Level Shifters/PAN5V.CS_02 -> /Panel Headers/HDR_CS_02_P1
- P10 pad 10: /Level Shifters/PAN5V.CS_18 -> /Panel Headers/HDR_CS_18_P10
- P10 pad 11: /Level Shifters/PAN5V.CS_19 -> /Panel Headers/HDR_CS_19_P10
- P10 pad 15: /Level Shifters/PAN5V.EXT_INT -> /Panel Headers/HDR_EXT_INT_P10
- P10 pad 4: /Level Shifters/PAN5V.SCK_1 -> /Panel Headers/HDR_SCK_1_P10
- P10 pad 5: /Level Shifters/PAN5V.MOSI_1 -> /Panel Headers/HDR_MOSI_1_P10
- P10 pad 6: /Level Shifters/PAN5V.MISO_1 -> /Panel Headers/HDR_MISO_1_P10
- P10 pad 7: /Level Shifters/PAN5V.CS_15 -> /Panel Headers/HDR_CS_15_P10
- P10 pad 8: /Level Shifters/PAN5V.CS_16 -> /Panel Headers/HDR_CS_16_P10
- P10 pad 9: /Level Shifters/PAN5V.CS_17 -> /Panel Headers/HDR_CS_17_P10
- P11 pad 10: /Level Shifters/PAN5V.CS_23 -> /Panel Headers/HDR_CS_23_P11
- P11 pad 11: /Level Shifters/PAN5V.CS_24 -> /Panel Headers/HDR_CS_24_P11
- P11 pad 15: /Level Shifters/PAN5V.EXT_INT -> /Panel Headers/HDR_EXT_INT_P11
- P11 pad 4: /Level Shifters/PAN5V.SCK_1 -> /Panel Headers/HDR_SCK_1_P11
- P11 pad 5: /Level Shifters/PAN5V.MOSI_1 -> /Panel Headers/HDR_MOSI_1_P11
- P11 pad 6: /Level Shifters/PAN5V.MISO_1 -> /Panel Headers/HDR_MISO_1_P11
- P11 pad 7: /Level Shifters/PAN5V.CS_20 -> /Panel Headers/HDR_CS_20_P11
- P11 pad 8: /Level Shifters/PAN5V.CS_21 -> /Panel Headers/HDR_CS_21_P11
- P11 pad 9: /Level Shifters/PAN5V.CS_22 -> /Panel Headers/HDR_CS_22_P11
- P12 pad 10: /Level Shifters/PAN5V.CS_28 -> /Panel Headers/HDR_CS_28_P12
- P12 pad 11: /Level Shifters/PAN5V.CS_29 -> /Panel Headers/HDR_CS_29_P12
- P12 pad 15: /Level Shifters/PAN5V.EXT_INT -> /Panel Headers/HDR_EXT_INT_P12
- P12 pad 4: /Level Shifters/PAN5V.SCK_1 -> /Panel Headers/HDR_SCK_1_P12
- P12 pad 5: /Level Shifters/PAN5V.MOSI_1 -> /Panel Headers/HDR_MOSI_1_P12
- P12 pad 6: /Level Shifters/PAN5V.MISO_1 -> /Panel Headers/HDR_MISO_1_P12
- P12 pad 7: /Level Shifters/PAN5V.CS_25 -> /Panel Headers/HDR_CS_25_P12
- P12 pad 8: /Level Shifters/PAN5V.CS_26 -> /Panel Headers/HDR_CS_26_P12
- P12 pad 9: /Level Shifters/PAN5V.CS_27 -> /Panel Headers/HDR_CS_27_P12
- P2 pad 10: /Level Shifters/PAN5V.CS_08 -> /Panel Headers/HDR_CS_08_P2
- P2 pad 11: /Level Shifters/PAN5V.CS_09 -> /Panel Headers/HDR_CS_09_P2
- P2 pad 15: /Level Shifters/PAN5V.EXT_INT -> /Panel Headers/HDR_EXT_INT_P2
- P2 pad 4: /Level Shifters/PAN5V.SCK_0 -> /Panel Headers/HDR_SCK_0_P2
- P2 pad 5: /Level Shifters/PAN5V.MOSI_0 -> /Panel Headers/HDR_MOSI_0_P2
- P2 pad 6: /Level Shifters/PAN5V.MISO_0 -> /Panel Headers/HDR_MISO_0_P2
- P2 pad 7: /Level Shifters/PAN5V.CS_05 -> /Panel Headers/HDR_CS_05_P2
- P2 pad 8: /Level Shifters/PAN5V.CS_06 -> /Panel Headers/HDR_CS_06_P2
- P2 pad 9: /Level Shifters/PAN5V.CS_07 -> /Panel Headers/HDR_CS_07_P2
- P3 pad 10: /Level Shifters/PAN5V.CS_13 -> /Panel Headers/HDR_CS_13_P3
- P3 pad 11: /Level Shifters/PAN5V.CS_14 -> /Panel Headers/HDR_CS_14_P3
- P3 pad 15: /Level Shifters/PAN5V.EXT_INT -> /Panel Headers/HDR_EXT_INT_P3
- P3 pad 4: /Level Shifters/PAN5V.SCK_0 -> /Panel Headers/HDR_SCK_0_P3
- P3 pad 5: /Level Shifters/PAN5V.MOSI_0 -> /Panel Headers/HDR_MOSI_0_P3
- P3 pad 6: /Level Shifters/PAN5V.MISO_0 -> /Panel Headers/HDR_MISO_0_P3
- P3 pad 7: /Level Shifters/PAN5V.CS_10 -> /Panel Headers/HDR_CS_10_P3
- P3 pad 8: /Level Shifters/PAN5V.CS_11 -> /Panel Headers/HDR_CS_11_P3
- P3 pad 9: /Level Shifters/PAN5V.CS_12 -> /Panel Headers/HDR_CS_12_P3
- P4 pad 10: /Level Shifters/PAN5V.CS_18 -> /Panel Headers/HDR_CS_18_P4
- P4 pad 11: /Level Shifters/PAN5V.CS_19 -> /Panel Headers/HDR_CS_19_P4
- P4 pad 15: /Level Shifters/PAN5V.EXT_INT -> /Panel Headers/HDR_EXT_INT_P4
- P4 pad 4: /Level Shifters/PAN5V.SCK_0 -> /Panel Headers/HDR_SCK_0_P4
- P4 pad 5: /Level Shifters/PAN5V.MOSI_0 -> /Panel Headers/HDR_MOSI_0_P4
- P4 pad 6: /Level Shifters/PAN5V.MISO_0 -> /Panel Headers/HDR_MISO_0_P4
- P4 pad 7: /Level Shifters/PAN5V.CS_15 -> /Panel Headers/HDR_CS_15_P4
- P4 pad 8: /Level Shifters/PAN5V.CS_16 -> /Panel Headers/HDR_CS_16_P4
- P4 pad 9: /Level Shifters/PAN5V.CS_17 -> /Panel Headers/HDR_CS_17_P4
- P5 pad 10: /Level Shifters/PAN5V.CS_23 -> /Panel Headers/HDR_CS_23_P5
- P5 pad 11: /Level Shifters/PAN5V.CS_24 -> /Panel Headers/HDR_CS_24_P5
- P5 pad 15: /Level Shifters/PAN5V.EXT_INT -> /Panel Headers/HDR_EXT_INT_P5
- P5 pad 4: /Level Shifters/PAN5V.SCK_0 -> /Panel Headers/HDR_SCK_0_P5
- P5 pad 5: /Level Shifters/PAN5V.MOSI_0 -> /Panel Headers/HDR_MOSI_0_P5
- P5 pad 6: /Level Shifters/PAN5V.MISO_0 -> /Panel Headers/HDR_MISO_0_P5
- P5 pad 7: /Level Shifters/PAN5V.CS_20 -> /Panel Headers/HDR_CS_20_P5
- P5 pad 8: /Level Shifters/PAN5V.CS_21 -> /Panel Headers/HDR_CS_21_P5
- P5 pad 9: /Level Shifters/PAN5V.CS_22 -> /Panel Headers/HDR_CS_22_P5
- P6 pad 10: /Level Shifters/PAN5V.CS_28 -> /Panel Headers/HDR_CS_28_P6
- P6 pad 11: /Level Shifters/PAN5V.CS_29 -> /Panel Headers/HDR_CS_29_P6
- P6 pad 15: /Level Shifters/PAN5V.EXT_INT -> /Panel Headers/HDR_EXT_INT_P6
- P6 pad 4: /Level Shifters/PAN5V.SCK_0 -> /Panel Headers/HDR_SCK_0_P6
- P6 pad 5: /Level Shifters/PAN5V.MOSI_0 -> /Panel Headers/HDR_MOSI_0_P6
- P6 pad 6: /Level Shifters/PAN5V.MISO_0 -> /Panel Headers/HDR_MISO_0_P6
- P6 pad 7: /Level Shifters/PAN5V.CS_25 -> /Panel Headers/HDR_CS_25_P6
- P6 pad 8: /Level Shifters/PAN5V.CS_26 -> /Panel Headers/HDR_CS_26_P6
- P6 pad 9: /Level Shifters/PAN5V.CS_27 -> /Panel Headers/HDR_CS_27_P6
- P7 pad 10: /Level Shifters/PAN5V.CS_03 -> /Panel Headers/HDR_CS_03_P7
- P7 pad 11: /Level Shifters/PAN5V.CS_04 -> /Panel Headers/HDR_CS_04_P7
- P7 pad 15: /Level Shifters/PAN5V.EXT_INT -> /Panel Headers/HDR_EXT_INT_P7
- P7 pad 4: /Level Shifters/PAN5V.SCK_1 -> /Panel Headers/HDR_SCK_1_P7
- P7 pad 5: /Level Shifters/PAN5V.MOSI_1 -> /Panel Headers/HDR_MOSI_1_P7
- P7 pad 6: /Level Shifters/PAN5V.MISO_1 -> /Panel Headers/HDR_MISO_1_P7
- P7 pad 7: /Level Shifters/PAN5V.CS_00 -> /Panel Headers/HDR_CS_00_P7
- P7 pad 8: /Level Shifters/PAN5V.CS_01 -> /Panel Headers/HDR_CS_01_P7
- P7 pad 9: /Level Shifters/PAN5V.CS_02 -> /Panel Headers/HDR_CS_02_P7
- P8 pad 10: /Level Shifters/PAN5V.CS_08 -> /Panel Headers/HDR_CS_08_P8
- P8 pad 11: /Level Shifters/PAN5V.CS_09 -> /Panel Headers/HDR_CS_09_P8
- P8 pad 15: /Level Shifters/PAN5V.EXT_INT -> /Panel Headers/HDR_EXT_INT_P8
- P8 pad 4: /Level Shifters/PAN5V.SCK_1 -> /Panel Headers/HDR_SCK_1_P8
- P8 pad 5: /Level Shifters/PAN5V.MOSI_1 -> /Panel Headers/HDR_MOSI_1_P8
- P8 pad 6: /Level Shifters/PAN5V.MISO_1 -> /Panel Headers/HDR_MISO_1_P8
- P8 pad 7: /Level Shifters/PAN5V.CS_05 -> /Panel Headers/HDR_CS_05_P8
- P8 pad 8: /Level Shifters/PAN5V.CS_06 -> /Panel Headers/HDR_CS_06_P8
- P8 pad 9: /Level Shifters/PAN5V.CS_07 -> /Panel Headers/HDR_CS_07_P8
- P9 pad 10: /Level Shifters/PAN5V.CS_13 -> /Panel Headers/HDR_CS_13_P9
- P9 pad 11: /Level Shifters/PAN5V.CS_14 -> /Panel Headers/HDR_CS_14_P9
- P9 pad 15: /Level Shifters/PAN5V.EXT_INT -> /Panel Headers/HDR_EXT_INT_P9
- P9 pad 4: /Level Shifters/PAN5V.SCK_1 -> /Panel Headers/HDR_SCK_1_P9
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Routing:
- added copper zone on In2.Cu, net +5V
- added copper zone on In1.Cu, net GND
Other:
- board outline added: 228.6 x 228.6 mm
- copper layers 4 -> 6

Commit message: Finished preliminary layout for new 12-12 teensy 4.1 arena.
Includes source termination resistors and schmitt trigger buffers.
Parts:
- C1, C10, C11, C12, C13, C14, C15, C16, C17, C18, C19, C2, C20, C21, C22, C23, C24, C25, C26, C27, C28, C29, C3, C30, C31, C32, C33, C34, C35, C36, C37, C38, C39, C4, C40, C41, C42, C43, C44, C45, C46, C47, C48, C49, C5, C50, C51, C52, C53, C54, C55, C56, C57, C58, C59, C6, C60, C61, C62, C63, C64, C65, C66, C67, C68, C69, C7, C70, C71, C72, C73, C74, C75, C76, C77, C78, C79, C8, C80, C81, C82, C83, C84, C85, C86, C87, C88, C89, C9, C90, C91, C92, C93, C94: footprint Capacitor_SMD:C_0603_1608Metric -> Capacitor_SMD:C_0402_1005Metric
- R10, R100, R101, R102, R103, R104, R105, R106, R107, R108, R109, R11, R110, R111, R112, R113, R114, R115, R116, R117, R118, R119, R12, R120, R121, R122, R123, R124, R125, R126, R127, R128, R129, R13, R130, R131, R132, R133, R134, R135, R136, R137, R138, R139, R14, R140, R141, R142, R143, R144, R145, R146, R147, R148, R149, R15, R150, R151, R152, R153, R154, R155, R156, R157, R158, R159, R16, R160, R161, R162, R163, R164, R165, R166, R167, R168, R169, R17, R170, R171, R172, R173, R174, R175, R176, R177, R178, R179, R18, R180, R181, R182, R183, R184, R185, R186, R187, R188, R189, R19, R190, R191, R192, R193, R194, R195, R196, R197, R198, R199, R20, R200, R201, R202, R203, R204, R205, R206, R207, R208, R209, R21, R210, R211, R212, R213, R214, R215, R216, R217, R218, R219, R22, R220, R221, R222, R223, R224, R225, R226, R227, R228, R229, R23, R230, R231, R232, R233, R234, R24, R25, R26, R27, R28, R29, R3, R30, R31, R32, R33, R34, R35, R36, R37, R38, R39, R4, R40, R41, R42, R43, R44, R45, R46, R47, R48, R49, R5, R50, R51, R52, R53, R54, R55, R56, R57, R58, R59, R6, R60, R61, R62, R63, R64, R65, R66, R67, R68, R69, R7, R70, R71, R72, R73, R74, R75, R76, R77, R78, R79, R8, R80, R81, R82, R83, R84, R85, R86, R87, R88, R89, R9, R90, R91, R92, R93, R94, R95, R96, R97, R98, R99: footprint Resistor_SMD:R_0603_1608Metric -> Resistor_SMD:R_0402_1005Metric
- moved C91 349.8 mm to (264.2, 217.5), turned to 150 degrees
- moved C92 347.7 mm to (260.5, 223.9), turned to 150 degrees
- moved C93 346.0 mm to (257.9, 228.4), turned to 150 degrees
- moved C94 344.3 mm to (255.1, 233.1), turned to 150 degrees
- moved C87 341.6 mm to (232.7, 255.4), turned to 120 degrees
- moved C54 340.0 mm to (264.4, 138.5), turned to -150 degrees
- moved R215 337.6 mm to (265.0, 216.2), turned to -30 degrees
- moved C53 336.9 mm to (261.7, 133.8), turned to -150 degrees
- moved C88 336.7 mm to (226.4, 259.0), turned to 120 degrees
- moved R216 336.3 mm to (263.4, 218.9), turned to -30 degrees
- moved R217 334.9 mm to (261.3, 222.4), turned to -30 degrees
- moved C52 334.1 mm to (259.0, 129.2), turned to -150 degrees
- moved R218 333.6 mm to (259.7, 225.3), turned to -30 degrees
- moved C89 332.8 mm to (221.8, 261.7), turned to 120 degrees
- moved R219 332.3 mm to (258.7, 227.0), turned to -30 degrees
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