File: development/arena_12-12/teensy4p1/teensy_arena_12-12_v0p1/panel_headers.kicad_sch (KiCad schematic)
At the start: 231 parts, among them P1 CONN15, P10 CONN15, P11 CONN15, P12 CONN15, P2 CONN15, P3 CONN15, P4 CONN15, P5 CONN15, P6 CONN15, P7 CONN15, P8 CONN15, P9 CONN15, Q1 MOSFET_NCHAN, U36 74LVC2G17, U37 74LVC2G17, U38 74LVC2G17, U39 74LVC2G17, U40 74LVC2G17, U41 74LVC2G17, U42 74LVC2G17, U43 74LVC2G17, U44 74LVC2G17, U45 74LVC2G17, U46 74LVC2G17, U47 74LVC2G17, U48 74LVC2G17, U49 74LVC2G17, U50 74LVC2G17, U51 74LVC2G17, U52 74LVC2G17, U53 74LVC2G17, U54 74LVC2G17, U55 74LVC2G17, U56 74LVC2G17, U57 74LVC2G17, U58 74LVC2G17, U59 74LVC2G17, U60 74LVC2G17, U61 74LVC2G17, U62 74LVC2G17, U63 74LVC2G17, U64 74LVC2G17, U65 74LVC2G17, U66 74LVC2G17, U67 74LVC2G17, U68 74LVC2G17, U69 74LVC2G17, U70 74LVC2G17, U71 74LVC2G17, U72 74LVC2G17, U73 74LVC2G17, U74 74LVC2G17, U75 74LVC2G17, U76 74LVC2G17, U77 74LVC2G17, U78 74LVC2G17, U79 74LVC2G17, U80 74LVC2G17, U81 74LVC2G17, U82 74LVC2G17, U83 74LVC2G17

Commit message: Finished hand route of 12-12 teensy arena. Finished route of 12-12 top.
Connections:
- net +3.3V is gone; now on net +5V: C47.1, C48.1, C49.1, C50.1, C51.1, C52.1, C53.1, C54.1, C55.1, C56.1, C57.1, C58.1, C59.1, C60.1, C61.1, C62.1, C63.1, C64.1, C65.1, C66.1, C67.1, C68.1, C69.1, C70.1, C71.1, C72.1, C73.1, C74.1, C75.1, C76.1, C77.1, C78.1, C79.1, C80.1, C81.1, C82.1, C83.1, C84.1, C85.1, C86.1, C87.1, C88.1, C89.1, C90.1, C91.1, C92.1, C93.1, C94.1, U36.5 (VCC), U37.5 (VCC), U38.5 (VCC), U39.5 (VCC), U40.5 (VCC), U41.5 (VCC), U42.5 (VCC), U43.5 (VCC), U44.5 (VCC), U45.5 (VCC), U46.5 (VCC), U47.5 (VCC), U48.5 (VCC), U49.5 (VCC), U50.5 (VCC), U51.5 (VCC), U52.5 (VCC), U53.5 (VCC), U54.5 (VCC), U55.5 (VCC), U56.5 (VCC), U57.5 (VCC), U58.5 (VCC), U59.5 (VCC), U60.5 (VCC), U61.5 (VCC), U62.5 (VCC), U63.5 (VCC), U64.5 (VCC), U65.5 (VCC), U66.5 (VCC), U67.5 (VCC), U68.5 (VCC), U69.5 (VCC), U70.5 (VCC), U71.5 (VCC), U72.5 (VCC), U73.5 (VCC), U74.5 (VCC), U75.5 (VCC), U76.5 (VCC), U77.5 (VCC), U78.5 (VCC), U79.5 (VCC), U80.5 (VCC), U81.5 (VCC), U82.5 (VCC), U83.5 (VCC)

Commit message: Finished initial verions of fab files for 12-12 teensy 4.1 arena. Need to check orientations.
Parts:
- R127, R128, R129, R130, R131, R132, R133, R134, R135, R136, R137, R138, R139, R140, R141, R142, R143, R144, R145, R146, R147, R148, R149, R150, R151, R152, R153, R154, R155, R156, R157, R158, R159, R160, R161, R162, R163, R164, R165, R166, R167, R168, R169, R170, R171, R172, R173, R174, R175, R176, R177, R178, R179, R180, R181, R182, R183, R184, R185, R186, R187, R188, R189, R190, R191, R192, R193, R194, R195, R196, R197, R198, R199, R200, R201, R202, R203, R204, R205, R206, R207, R208, R209, R210, R211, R212, R213, R214, R215, R216, R217, R218, R219, R220, R221, R222, R223, R224, R225, R226, R227, R228, R229, R230, R231, R232, R233, R234: value 68 -> 33
