File: development/arena_12-12/top/arena_top_12-12/layout_tool/modified_arena_top_12-12.kicad_pcb (KiCad board)
At the start: 6 copper layers, 228.6 x 228.6 mm, 41 parts, among them J4 Barrel_Jack, P1 CONN15, P10 CONN15, P11 CONN15, P12 CONN15, P2 CONN15, P3 CONN15, P4 CONN15, P5 CONN15, P6 CONN15, P7 CONN15, P8 CONN15, P9 CONN15

Commit message: Finished hand route of 12-12 teensy arena. Finished route of 12-12 top.
Parts:
- P1, P10, P11, P12, P2, P3, P4, P5, P6, P7, P8, P9: moved to B.Cu
- moved C14 352.5 mm to (254.4, 113.0), turned to -60 degrees
- moved C24 330.3 mm to (272.2, 211.8), turned to -120 degrees
- moved C15 324.4 mm to (211.8, 83.4), turned to -30 degrees
- moved C23 305.7 mm to (242.6, 254.4), turned to -150 degrees
- moved C22 268.1 mm to (195.6, 276.5), turned to 180 degrees
- moved C16 262.2 mm to (160.0, 79.1)
- moved C21 221.0 mm to (143.8, 272.2), turned to 150 degrees
- moved C17 214.5 mm to (113.0, 101.2), turned to 30 degrees
- moved C20 174.5 mm to (101.2, 242.6), turned to 120 degrees
- moved C18 173.7 mm to (83.4, 143.8), turned to 60 degrees
- moved C19 147.1 mm to (79.1, 195.6), turned to 90 degrees
- moved C10 2.79 mm to (194.3, 270.1)
- moved C4 2.79 mm to (161.3, 85.5)
- moved C7 2.79 mm to (85.5, 194.3)
- moved C2 2.79 mm to (249.4, 117.3)
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